File: schematics/anchor/anchor.kicad_sch (KiCad schematic)
At the start: 61 parts, among them J16 Screw_Terminal_01x01, J18 Screw_Terminal_01x01, J7 IEC_60320_C14_Receptacle, M1 Motor_X0, M10 Motor_Z2, M2 Motor_Y0, M26 Fan, M27 Fan, M3 Fan, M4 Fan, M5 Motor_X1, M6 Motor_Y1, M7 Motor_E0, M8 Motor_Z0, M9 Motor_Z1, SW2 SW_DPST, SW5 Thermostat, T1 Meanwell_UHP-200-48, T2 Meanwell_UHP-200-24, T5 Meanwell_UHP-200-5, U1 Phoenix_Contact_PTFIX_6x2, U10 Beacon_Regulator, U11 Phoenix_Contact_PTFIX_6x2, U12 Schneider_Electric_DPE25BL, U13 Phoenix_Contact_PTFIX_12x2, U14 Schneider_Electric_DPE25BL, U19 BTT_TMC5160T_Plus, U2 Phoenix_Contact_PTFIX_6x2, U22 Schneider_Electric_DPE25G7, U23 Raspberry_Pi, U24 Adafruit_Feather_Relay, U3 Phoenix_Contact_PTFIX_6x2, U4 Schneider_Electric_DPE25BL, U5 Crydom_D2440_SPST_SSR-NO, U6 Crydom_D2440_SPST_SSR-NO, U7 Schneider_Electric_DPE25BL, U8 Beacon_Eddy_Scanner, U9 Phoenix_Contact_PTFIX_6x2

Commit message: Split schematic to sections
Parts:
- removed D8: D, symbol Device:D
- removed D9: D_Zener, symbol Device:D_Zener
- removed F4: Fuse, symbol Device:Fuse
- removed M1: Motor_X0, symbol Motor:Stepper_Motor_bipolar
- removed M10: Motor_Z2, symbol Motor:Stepper_Motor_bipolar
- removed M2: Motor_Y0, symbol Motor:Stepper_Motor_bipolar
- removed M5: Motor_X1, symbol Motor:Stepper_Motor_bipolar
- removed M6: Motor_Y1, symbol Motor:Stepper_Motor_bipolar
- removed M7: Motor_E0, symbol Motor:Stepper_Motor_bipolar
- removed M8: Motor_Z0, symbol Motor:Stepper_Motor_bipolar
- removed M9: Motor_Z1, symbol Motor:Stepper_Motor_bipolar
- removed R15, R17: 24VDC 100W Heater, symbol Device:Heater
- removed TH14, TH16: Thermistor_PTC, symbol Device:Thermistor_PTC
- removed U12, U14: Schneider_Electric_DPE25BL, symbol jmatt:Schneider_Electric_DPE25BL
- removed U16: ~, symbol jmatt:Murrelektronik_Diode_Zener_Suppressor
- removed U8: Beacon_Eddy_Scanner, symbol jmatt:Beacon_Eddy_Scanner
- added F10, F8: XXA, symbol Device:Fuse
- added F16, F17, F19, F21: Thermal_Fuse, symbol jmatt:Thermal_Fuse
- added F20, F6, F7: Fuse, symbol Device:Fuse
- added J10, J8: IEC_60320_C14_Receptacle, symbol Connector:IEC_60320_C14_Receptacle
- added J17, J19: Screw_Terminal_01x01, symbol Connector:Screw_Terminal_01x01
- added M11, M12: Fan, symbol Motor:Fan_3pin
- added M21, M23, M24, M25: Motor_E0, symbol Motor:Stepper_Motor_bipolar
- added M22: Motor_X0, symbol Motor:Stepper_Motor_bipolar
- added M28, M29: Fan, symbol Motor:Fan
- added M30: Motor_Z0, symbol Motor:Stepper_Motor_bipolar
- added M31: Motor_Z1, symbol Motor:Stepper_Motor_bipolar
- added M32: Motor_Z2, symbol Motor:Stepper_Motor_bipolar
- added M33: Motor_CPAP, symbol Motor:Stepper_Motor_bipolar
- added R16: 120VAC 750W Heater, symbol Device:Heater
- added R21: 120VAC 250W Heater x2, symbol Device:Heater
- added R22: 120VAC 500W Heater, symbol Device:Heater
- added R25: 24VDC 100W Heater, symbol Device:Heater
- added SW3, SW7: SW_DPST, symbol Switch:SW_DPST
- added T16, T3: Meanwell_UHP-200-48, symbol jmatt:UHP-200-24
- added T17, T4: Meanwell_UHP-200-24, symbol jmatt:UHP-200-24
- added T6, T7: Meanwell_UHP-200-5, symbol jmatt:UHP-200-24
- added TH10, TH14, TH16, TH17, TH18, TH19, TH21, TH22, TH23, TH24, TH25, TH7, TH8, TH9: Thermistor_NTC, symbol Device:Thermistor_NTC
- added TH12, TH15, TH20: Thermistor_PTC, symbol Device:Thermistor_PTC
- added U20, U26: Crydom_D2440_SPST_SSR-NO, symbol jmatt:Crydom_D2440_SPST_SSR-NO
- added U21, U27, U46: Schneider_Electric_DPE25BL, symbol jmatt:Schneider_Electric_DPE25BL
- added U25, U28, U47: ~, symbol jmatt:Murrelektronik_Diode_Zener_Suppressor
- added U29: ~, symbol jmatt:SW_SPST_NC_Temperature_Flipped
- added U32, U41: Schneider_Electric_DPE25G7, symbol jmatt:Schneider_Electric_DPE25G7
- added U34, U40: ~, symbol jmatt:Murrelektronik_26183_Varistor_Suppressor
- added U36, U39: Adafruit_Feather_Relay, symbol jmatt:Adafruit_Feather_Relay
- added U45: Beacon_Eddy_Scanner, symbol jmatt:Beacon_Eddy_Scanner
Connections:
- net Earth_Protective: now also J10.3 (PE), J8.3 (PE)
- net GND: now also U10.1 (GND), T16.1 (V-), T17.1 (V-), T3.1 (V-), T4.1 (V-), T6.1 (V-), T7.1 (V-), U36.4 (GND), U39.4 (GND), U45.1 (GND)
- net at U3.4: no longer T1.2 (V+)
- net at U13.11: no longer T2.3 (PE)
- net BEACON_D-: now reaches U10.2 (D+)
- net BEACON_D-: now also U45.3 (D-)
- net BEACON_D+: now reaches U10.3 (D-)
- net BEACON_D+: now also U45.2 (D+)
- net VBUS: now reaches U10.4 (+5VDC)
- net VBUS: now also U45.4 (+5VDC)
- net at J7.2 (N): now also SW2.2
- net at T5.1 (V-), U24.4 (GND): no longer U23. (+5VDC)
- net at T5.2 (V+), U24.2 (+5VDC): no longer U23. (+5VDC)
- net at U24.5 (RELAY): no longer U23.16 (GPIO23)
- net at T1.1 (V-): now also U9.4
- net at T2.1 (V-): now also U9.5
- new net: F16.1, U20.2 (AC)
- new net: F16.2, R16.1
- new net: F10.2, J10.1 (L)
- new net: J10.2 (N), SW7.1
- new net: F7.1, U27.2 (2/T1)
- new net: R21.2, R22.2, U27.4 (4/T2)
- new net: F6.1, U21.2 (2/T1)
- new net: R16.2, U21.4 (4/T2)
- new net: F20.1, U46.2 (2/T1)
- new net: F20.2, R25.1
- new net: F19.1, F7.2
- new net: U39., U40.1, U41.A1
- new net: SW7.4, T7.1 (V-), U39., U41.1 (1/L1)
- new net: F21.1, U29.2
- new net: F21.2, U26.2 (AC)
- new net: R21.1, R22.1, U29.1
- new net: F10.1, SW7.3
- new net: SW3.1, T6.2 (V+), U32.3 (3/L2), U32.A2, U34.2
- new net: J8.2 (N), SW3.2
- new net: SW3.3, T6.1 (V-), U32.1 (1/L1), U36.
- new net: F8.1, SW3.4
- new net: F17.2, U20.1 (AC)
- new net: F17.1, F6.2
- new net: SW7.2, T7.2 (V+), U40.2, U41.3 (3/L2), U41.A2
- new net: U32.A1, U34.1, U36.
- new net: F19.2, U26.1 (AC)
- new net: F8.2, J8.1 (L)
- new net: R25.2, U46.4 (4/T2)
- new net +24V: T17.2 (V+), T4.2 (V+)
- new net +48V: T16.2 (V+), T3.2 (V+)
- new net +5V: T6.2 (V+), T7.2 (V+), U36.2 (+5VDC), U39.2 (+5VDC)
- new net 120VAC_L_SWITCHED: T16.1 (V-), T17.1 (V-), U21.1 (1/L1), U27.1 (1/L1), U41.2 (2/T1)
- new net 120VAC_L_Switched: T3.1 (V-), T4.1 (V-), U32.2 (2/T1)
- new net 120VAC_N_SWITCHED: T16.2 (V+), T17.2 (V+), U21.3 (3/L2), U27.3 (3/L2), U41.4 (4/T2)
- new net 120VAC_N_Switched: T3.2 (V+), T4.2 (V+), U32.4 (4/T2)
- new net BED_CONTACTOR+: U21.A1 (A1+), U25.1 (+)
- new net BED_CONTACTOR-: U21.A2 (A2-), U25.2 (-)
- new net BED_FAN+: M28.1 (+), M29.1 (+)
- new net BED_FAN-: M28.2 (-), M29.2 (-)
- new net BED_HEATER+: U20.3 (IN+)
- new net BED_HEATER-: U20.4 (IN-)
- new net BED_THERM: TH12.1, TH12.2
- new net CHASSIS: J10.3 (PE), J17.1 (Pin_1), J19.1 (Pin_1), J8.3 (PE), T16.3 (PE), T17.3 (PE), T3.3 (PE), T4.3 (PE), T6.3 (PE), T7.3 (PE), U20.5 (PE), U26.5 (PE)
- new net CH_CONTACTOR+: U27.A1 (A1+), U28.1 (+)
- new net CH_CONTACTOR-: U27.A2 (A2-), U28.2 (-)
- new net CH_FAN+: M11.2 (+), M12.2 (+)
- new net CH_FAN-: M11.1 (-), M12.1 (-)
- new net CH_FAN_ALARM: M11.3 (Alarm), M12.3 (Alarm)
- new net CH_HEATER+: U26.3 (IN+)
- new net CH_HEATER-: U26.4 (IN-)
- new net CH_THERM: TH15.1, TH15.2
- new net HE_CONTACTOR+: U46.A1 (A1+), U47.1 (+)
- new net HE_CONTACTOR-: U46.A2 (A2-), U47.2 (-)
- new net HE_HEATER+: U46.1 (1/L1)
- new net HE_HEATER-: U46.3 (3/L2)
- new net HE_THERM: TH20.1, TH20.2
- new net LOWER_CH_THERM_0: TH23.1, TH23.2
- new net LOWER_CH_THERM_1: TH24.1, TH24.2
- new net LOWER_CH_THERM_2: TH25.1, TH25.2
- new net MOTOR_CPAP_A1: M33.4
- new net MOTOR_CPAP_A2: M33.3
- new net MOTOR_CPAP_B1: M33.1
- new net MOTOR_CPAP_B2: M33.2 (-)
- new net MOTOR_E0_A1: M21.4
- new net MOTOR_E0_A2: M21.3
- new net MOTOR_E0_B1: M21.1
- new net MOTOR_E0_B2: M21.2 (-)
- new net MOTOR_E0_THERM: TH7.1, TH7.2
- new net MOTOR_X0_A1: M22.4
- new net MOTOR_X0_A2: M22.3
- new net MOTOR_X0_B1: M22.1
- new net MOTOR_X0_B2: M22.2 (-)
- new net MOTOR_X0_THERM: TH8.1, TH8.2
- new net MOTOR_X1_A1: M24.4
- new net MOTOR_X1_A2: M24.3
- new net MOTOR_X1_B1: M24.1
- new net MOTOR_X1_B2: M24.2 (-)
- new net MOTOR_X1_THERM: TH10.1, TH10.2
- new net MOTOR_Y0_A1: M23.4
- new net MOTOR_Y0_A2: M23.3
- new net MOTOR_Y0_B1: M23.1
- new net MOTOR_Y0_B2: M23.2 (-)
- new net MOTOR_Y0_THERM: TH9.1, TH9.2
- new net MOTOR_Y1_A1: M25.4
- new net MOTOR_Y1_A2: M25.3
- new net MOTOR_Y1_B1: M25.1
- new net MOTOR_Y1_B2: M25.2 (-)
- new net MOTOR_Y1_THERM: TH14.1, TH14.2
- new net MOTOR_Z0_A1: M30.4
- new net MOTOR_Z0_A2: M30.3
- new net MOTOR_Z0_B1: M30.1
- new net MOTOR_Z0_B2: M30.2 (-)
- new net MOTOR_Z0_THERM: TH16.1, TH16.2
- new net MOTOR_Z1_A1: M31.4
- new net MOTOR_Z1_A2: M31.3
- new net MOTOR_Z1_B1: M31.1
- new net MOTOR_Z1_B2: M31.2 (-)
- new net MOTOR_Z1_THERM: TH17.1, TH17.2
- new net MOTOR_Z2_A1: M32.4
- new net MOTOR_Z2_A2: M32.3
- new net MOTOR_Z2_B1: M32.1
- new net MOTOR_Z2_B2: M32.2 (-)
- new net MOTOR_Z2_THERM: TH18.1, TH18.2
- new net Pi_Relay: U23.16 (GPIO23), U36.5 (RELAY), U39.5 (RELAY)
- new net UPPER_CH_THERM_0: TH19.1, TH19.2
- new net UPPER_CH_THERM_1: TH21.1, TH21.2
- new net UPPER_CH_THERM_2: TH22.1, TH22.2
- no-connect marks 20 -> 32
Other:
- note added: "Power"
- note added: "TODO * chamber circulation fans * chamber camera * chamber LEDs * electronics bay thermistors * electronics bay fans * electronics bay LEDs * microcontrollers * stepper drivers * CPAP stuff * front panel status LEDS * front panel display"
- moved on the sheet: U10, U19, U23

Commit message: Add LEDs; fix thermistor naming scheme to allow DRC
Parts:
- added M? (x4): Fan_4pin, symbol Motor:Fan_4pin
- added SW? (x4): SW_DPST, symbol Switch:SW_DPST
- added TH1, TH2: Thermistor_NTC, symbol Device:Thermistor_NTC
- added U? (x8): Daylight_On_A_Stick_XXL, symbol jmatt:Daylight_On_A_Stick_XXL
- added U? (x8): Disco_On_A_Stick_XXL, symbol jmatt:Disco_On_A_Stick_XXL
- renumbered F16 to F?, F18 to F?, F20 to F?, F7 to F?, F21 to F?, F5 to F?, F10 to F?, F14 to F?, F17 to F?, F6 to F?, F19 to F?, F8 to F?, F3 to F?, F2 to F?, F13 to F?, F15 to F?, J10 to J?, J7 to J?, J19 to J?, J17 to J?, J8 to J?, J18 to J?, J16 to J?, M29 to M?, M27 to M?, M33 to M?, M21 to M?, M30 to M?, M32 to M?, M12 to M?, M22 to M?, M25 to M?, M4 to M?, M3 to M?, M23 to M?, M28 to M?, M24 to M?, M11 to M?, M31 to M?, M26 to M?, R21 to R?, R16 to R?, R20 to R?, R14 to R?, R22 to R?, R19 to R?, R25 to R?, SW3 to SW?, SW2 to SW?, SW7 to SW?, SW5 to SW?, T16 to T?, T6 to T?, T5 to T?, T7 to T?, T17 to T?, T1 to T?, T4 to T?, T2 to T?, T3 to T?, TH16 to TH?, TH17 to TH?, TH22 to TH?, TH21 to TH?, TH24 to TH?, TH10 to TH?, TH14 to TH?, TH25 to TH?, TH23 to TH?, TH20 to TH?, TH19 to TH?, TH8 to TH?, TH13 to TH?, TH11 to TH?, TH9 to TH?, TH12 to TH?, TH15 to TH?, TH18 to TH?, TH7 to TH?, U47 to U?, U22 to U?, U3 to U?, U19 to U?, U27 to U?, U21 to U?, U2 to U?, U13 to U?, U39 to U?, U18 to U?, U11 to U?, U10 to U?, U20 to U?, U7 to U?, U29 to U?, U25 to U?, U4 to U?, U1 to U?, U40 to U?, U36 to U?, U26 to U?, U32 to U?, U45 to U?, U15 to U?, U6 to U?, U23 to U?, U46 to U?, U5 to U?, U24 to U?, U34 to U?, U9 to U?, U41 to U?, U28 to U?, U17 to U?
Connections:
- net +5V: now also SW?.3, SW?.3
- net GND: now also U?.3 (GND), U?.3 (GND)
- net UPPER_CH_THERM_0: now also TH1.1, TH1.2; no longer TH?.1, TH?.2
- net UPPER_CH_THERM_1: now also TH2.1, TH2.2; no longer TH?.1, TH?.2
- net at J?.1 (L): now also F?.2
- net at J?.2 (N): now also SW?.1
- net at U?.: now also SW?.4, T?.1 (V-), U?.1 (1/L1)
- net at J?.2 (N): now also SW?.2
- net at U?.: now also U?.1, U?.A1
- net at T?.1 (V-): now also U?.4
- net at T?.1 (V-): now also U?.5
- net BED_THERM renamed BED_THERM_0
- net BED_THERM_0: no longer TH?.1
- net CH_THERM renamed CH_THERM_0
- net CH_THERM_0: no longer TH?.2
- net HE_THERM renamed HE_THERM_0
- net HE_THERM_0: no longer TH?.2
- net LOWER_CH_THERM_0 renamed LOWER_CH_THERM_0_0
- net LOWER_CH_THERM_0_0: no longer TH?.2
- net LOWER_CH_THERM_1 renamed LOWER_CH_THERM_1_0
- net LOWER_CH_THERM_1_0: no longer TH?.2
- net LOWER_CH_THERM_2 renamed LOWER_CH_THERM_2_0
- net LOWER_CH_THERM_2_0: no longer TH?.2
- net MOTOR_E0_THERM renamed MOTOR_E0_THERM_0
- net MOTOR_E0_THERM_0: no longer TH?.2
- net MOTOR_X0_THERM renamed MOTOR_X0_THERM_0
- net MOTOR_X0_THERM_0: no longer TH?.2
- net MOTOR_X1_THERM renamed MOTOR_X1_THERM_0
- net MOTOR_X1_THERM_0: no longer TH?.2
- net MOTOR_Y0_THERM renamed MOTOR_Y0_THERM_0
- net MOTOR_Y0_THERM_0: no longer TH?.2
- net MOTOR_Y1_THERM renamed MOTOR_Y1_THERM_0
- net MOTOR_Y1_THERM_0: no longer TH?.2
- net MOTOR_Z0_THERM renamed MOTOR_Z0_THERM_0
- net MOTOR_Z0_THERM_0: no longer TH?.2
- net MOTOR_Z1_THERM renamed MOTOR_Z1_THERM_0
- net MOTOR_Z1_THERM_0: no longer TH?.2
- net MOTOR_Z2_THERM renamed MOTOR_Z2_THERM_0
- net MOTOR_Z2_THERM_0: no longer TH?.2
- net UPPER_CH_THERM_2 renamed UPPER_CH_THERM_2_0
- net UPPER_CH_THERM_2_0: no longer TH?.2
- new net: SW?.4, U?.1 (+24VDC) (x2)
- new net: SW?.2, U?.2 (GND) (x2)
- new net: U?.1 (+24VDC), U?.3 (+24VDC) (x6)
- new net: U?.2 (GND), U?.4 (GND) (x6)
- new net: U?.1 (+5VDC), U?.4 (+5VDC) (x6)
- new net: U?.2 (DIN), U?.5 (DOUT) (x6)
- new net: U?.3 (GND), U?.6 (GND) (x6)
- new net: SW?.4, U?.1 (+5VDC) (x2)
- new net: SW?.2, U?.2 (DIN) (x2)
- new net BED_THERM_1: TH?.1
- new net CHAMBER_LED+: SW?.3
- new net CHAMBER_LED-: SW?.1
- new net CHAMBER_NEO: SW?.1
- new net CH_THERM_1: TH?.2
- new net EBAY_FAN+: M?.2 (+), M?.2 (+), M?.2 (+), M?.2 (+)
- new net EBAY_FAN-: M?.1 (-), M?.1 (-), M?.1 (-), M?.1 (-)
- new net EBAY_FAN_PWM: M?.4 (PWM), M?.4 (PWM), M?.4 (PWM), M?.4 (PWM)
- new net EBAY_FAN_TACH: M?.3 (Tacho), M?.3 (Tacho), M?.3 (Tacho), M?.3 (Tacho)
- new net EBAY_LED+: SW?.3
- new net EBAY_LED-: SW?.1
- new net EBAY_NEO: SW?.1
- new net HE_THERM_1: TH?.2
- new net LOWER_CH_THERM_0_1: TH?.2
- new net LOWER_CH_THERM_1_1: TH?.2
- new net LOWER_CH_THERM_2_1: TH?.2
- new net MOTOR_E0_THERM_1: TH?.2
- new net MOTOR_X0_THERM_1: TH?.2
- new net MOTOR_X1_THERM_1: TH?.2
- new net MOTOR_Y0_THERM_1: TH?.2
- new net MOTOR_Y1_THERM_1: TH?.2
- new net MOTOR_Z0_THERM_1: TH?.2
- new net MOTOR_Z1_THERM_1: TH?.2
- new net MOTOR_Z2_THERM_1: TH?.2
- new net UPPER_CH_THERM_0_0: TH?.1
- new net UPPER_CH_THERM_0_1: TH?.2
- new net UPPER_CH_THERM_1_0: TH?.1
- new net UPPER_CH_THERM_1_1: TH?.2
- new net UPPER_CH_THERM_2_1: TH?.2
- no-connect marks 32 -> 42
Other:
- note added: "TODO * chamber circulation fans * chamber camera * electronics bay thermistors * microcontrollers * stepper drivers * CPAP fan * CPAP flap * front panel status LEDS * front panel display * water cooling?"
- note removed: "TODO * chamber circulation fans * chamber camera * chamber LEDs * electronics bay thermistors * electronics bay fans * electronics bay LEDs * microcontrollers * stepper drivers * CPAP stuff * front panel status LEDS * front panel display"

Commit message: Add octopus symbol
Parts:
- removed F? (x4): Thermal_Fuse, symbol jmatt:Thermal_Fuse
- removed F? (x2): XXA, symbol Device:Fuse
- removed F? (x2): Fuse, symbol Device:Fuse
- removed J? (x2): IEC_60320_C14_Receptacle, symbol Connector:IEC_60320_C14_Receptacle
- removed J? (x2): Screw_Terminal_01x01, symbol Connector:Screw_Terminal_01x01
- removed M? (x2): Fan, symbol Motor:Fan
- removed M? (x4): Fan_4pin, symbol Motor:Fan_4pin
- removed M? (x2): Fan, symbol Motor:Fan_3pin
- removed R?: 120VAC 250W Heater x2, symbol Device:Heater
- removed R?: 120VAC 750W Heater, symbol Device:Heater
- removed R?: 120VAC 500W Heater, symbol Device:Heater
- removed SW? (x2): SW_DPST, symbol Switch:SW_DPST
- removed SW?: Thermostat, symbol jmatt:SW_SPST_NC_Temperature
- removed T? (x2): Meanwell_UHP-200-5, symbol jmatt:UHP-200-24
- removed T? (x2): Meanwell_UHP-200-48, symbol jmatt:UHP-200-24
- removed T? (x2): Meanwell_UHP-200-24, symbol jmatt:UHP-200-24
- removed TH? (x2): Thermistor_PTC, symbol Device:Thermistor_PTC
- removed U? (x2): Schneider_Electric_DPE25G7, symbol jmatt:Schneider_Electric_DPE25G7
- removed U? (x5): Phoenix_Contact_PTFIX_6x2, symbol jmatt:Phoenix_Contact_PTFIX_6x2
- removed U?: Phoenix_Contact_PTFIX_12x2, symbol jmatt:Phoenix_Contact_PTFIX_12x2
- removed U? (x2): ~, symbol jmatt:Murrelektronik_26183_Varistor_Suppressor
- removed U?: Beacon_Regulator, symbol jmatt:Beacon_Regulator
- removed U? (x2): Schneider_Electric_DPE25BL, symbol jmatt:Schneider_Electric_DPE25BL
- removed U? (x2): Adafruit_Feather_Relay, symbol jmatt:Adafruit_Feather_Relay
- removed U? (x2): ~, symbol jmatt:Murrelektronik_Diode_Zener_Suppressor
- removed U? (x2): Crydom_D2440_SPST_SSR-NO, symbol jmatt:Crydom_D2440_SPST_SSR-NO
- added M1, M2: Crossflow_Fan, symbol Motor:Fan
- added M3, M4, M5, M6: Fan_4pin, symbol Motor:Fan_4pin
- added SW1, SW2: SW_SPST, symbol Switch:SW_SPST
- added U1: e-CAM20_CU0230, symbol jmatt:USB_Camera
- added U2: OLED_HDMI_USB_Display, symbol jmatt:OLED_HDMI_USB_Display
- added U3: Overhub_7-Port_USB_3.0_MTT_Hub, symbol jmatt:Overhub_7-Port_USB_3.0_MTT_Hub
- added U4: Beacon_Regulator, symbol jmatt:Beacon_Regulator
- added U5: BTT_Octopus_Max_EZ, symbol jmatt:BTT_Octopus_Max_EZ
- added U6, U7, U8, U9: 5160T_Plus, symbol jmatt:BTT_TMC5160T_Plus
- M?: value Motor_CPAP -> Motor_CPAP_Flap
- U?: value BTT_TMC5160T_Plus -> 5160T_Plus
Connections:
- net 48VDC is gone; now on net +48V: U?.6 (+)
- net +24V: now also U5. (GND)
- net +48V: now also U6.6 (+), U7.6 (+), U8.6 (+), U9.6 (+)
- net +5V: now also U?. (+5VDC), U3.1 (+5VDC), U5. (GND)
- net BEACON_D+: now also U4.2 (D+)
- net BEACON_D-: now also U4.3 (D-)
- net EBAY_FAN+: now also M3.2 (+), M4.2 (+), M5.2 (+), M6.2 (+), U5. (GND)
- net EBAY_FAN-: now also M3.1 (-), M4.1 (-), M5.1 (-), M6.1 (-), U5. (GND)
- net EBAY_FAN_PWM: now also M3.4 (PWM), M4.4 (PWM), M5.4 (PWM), M6.4 (PWM), U5. (GND)
- net EBAY_FAN_TACH: now also M3.3 (Tacho), M4.3 (Tacho), M5.3 (Tacho), M6.3 (Tacho), U5. (GND)
- net GND: now also U?. (+5VDC), SW1.1 (A), SW2.1 (A), U1.4 (GND), U2.4 (GND), U3.2 (GND), U5. (GND), U6.5 (-), U7.5 (-), U8.5 (-), U9.5 (-); no longer U?.1 (GND)
- net MOTOR_E0_A1: now also U9.3 (A1)
- net MOTOR_E0_A2: now also U9.4 (A2)
- net MOTOR_E0_B1: now also U9.1 (B1)
- net MOTOR_E0_B2: now also U9.2 (B2)
- net MOTOR_X0_A1: now also U?.3 (A1)
- net MOTOR_X0_A2: now also U?.4 (A2)
- net MOTOR_X0_B1: now also U?.1 (B1)
- net MOTOR_X0_B2: now also U?.2 (B2)
- net MOTOR_X1_A1: now also U7.3 (A1)
- net MOTOR_X1_A2: now also U7.4 (A2)
- net MOTOR_X1_B1: now also U7.1 (B1)
- net MOTOR_X1_B2: now also U7.2 (B2)
- net MOTOR_Y0_A1: now also U6.3 (A1)
- net MOTOR_Y0_A2: now also U6.4 (A2)
- net MOTOR_Y0_B1: now also U6.1 (B1)
- net MOTOR_Y0_B2: now also U6.2 (B2)
- net MOTOR_Y1_A1: now also U8.3 (A1)
- net MOTOR_Y1_A2: now also U8.4 (A2)
- net MOTOR_Y1_B1: now also U8.1 (B1)
- net MOTOR_Y1_B2: now also U8.2 (B2)
- net MOTOR_Z0_A1: now also U5. (GND)
- net MOTOR_Z0_A2: now also U5. (GND)
- net MOTOR_Z0_B1: now also U5. (GND)
- net MOTOR_Z0_B2: now also U5. (GND)
- net MOTOR_Z1_A1: now also U5. (GND)
- net MOTOR_Z1_A2: now also U5. (GND)
- net MOTOR_Z1_B1: now also U5. (GND)
- net MOTOR_Z1_B2: now also U5. (GND)
- net MOTOR_Z2_A1: now also U5. (GND)
- net MOTOR_Z2_A2: now also U5. (GND)
- net MOTOR_Z2_B1: now also U5. (GND)
- net MOTOR_Z2_B2: now also U5. (GND)
- net VBUS: now also U1.1 (+5VDC), U2.1 (+5VDC); no longer U?.4 (+5VDC)
- net at U?.: now also U5. (GND)
- net at J?.1 (L): now also F?.2
- net at J?.2 (N): now also SW?.1
- net at U?.: now also SW?.4, T?.1 (V-), U?.1 (1/L1)
- net MOTOR_CPAP_A1 renamed MOTOR_CPAP_FLAP_A1
- net MOTOR_CPAP_FLAP_A1: now also U5. (GND)
- net MOTOR_CPAP_A2 renamed MOTOR_CPAP_FLAP_A2
- net MOTOR_CPAP_FLAP_A2: now also U5. (GND)
- net MOTOR_CPAP_B1 renamed MOTOR_CPAP_FLAP_B1
- net MOTOR_CPAP_FLAP_B1: now also U5. (GND)
- net MOTOR_CPAP_B2 renamed MOTOR_CPAP_FLAP_B2
- net MOTOR_CPAP_FLAP_B2: now also U5. (GND)
- net UPPER_CH_THERM_0 renamed EBAY_INTAKE_THERM_0
- net EBAY_INTAKE_THERM_0: no longer TH1.2
- net UPPER_CH_THERM_1 renamed EBAY_EXHAUST_THERM_0
- net EBAY_EXHAUST_THERM_0: no longer TH2.2
- new net: U3. (D-), U4.5
- new net: U3. (D-), U4.6
- new net: U3. (D-), U4.7
- new net: U3. (D-), U4.8
- new net: U3.3 (GND), U?. (+5VDC)
- new net: U3.4 (D-), U?. (+5VDC)
- new net: U3.5 (D+), U?. (+5VDC)
- new net: U3.6 (VBUS), U?. (+5VDC)
- new net: U5. (GND), U9.
- new net: U5. (GND), U8.
- new net: U5. (GND), U7.
- new net: U5. (GND), U6.
- new net BEACON_GND: U4.1 (GND), U?.1 (GND)
- new net BEACON_VBUS: U4.4 (+5VDC), U?.4 (+5VDC)
- new net CAMERA_D+: U1.2 (D+), U3. (D-)
- new net CAMERA_D-: U1.3 (D-), U3. (D-)
- new net CH_CIRC_FAN+: M1.1 (+), M2.1 (+)
- new net CH_CIRC_FAN-: M1.2 (-), M2.2 (-)
- new net DISPLAY_D+: U2.2 (D+), U3. (D-)
- new net DISPLAY_D-: U2.3 (D-), U3. (D-)
- new net DISPLAY_HDMI: U2.5 (HDMI), U?. (+5VDC)
- new net EBAY_EXHAUST_THERM_1: TH2.2
- new net EBAY_INTAKE_THERM_1: TH1.2
- new net OCTOPUS_D+: U3. (D-), U5. (GND)
- new net OCTOPUS_D-: U3. (D-), U5. (GND)
- new net THERMX_D+: U3. (D-)
- new net THERMX_D-: U3. (D-)
- new net X_ENDSTOP: SW1.2 (B), U5. (GND)
- new net Y_ENDSTOP: SW2.2 (B), U5. (GND)
- no-connect marks 42 -> 87
Other:
- note added: "Raspberry Pi"
- note added: "TODO * microcontrollers * stepper drivers * CPAP fan * front panel status LEDS * water cooling? * toolhead leds?"
- note removed: "TODO * chamber circulation fans * chamber camera * electronics bay thermistors * microcontrollers * stepper drivers * CPAP fan * CPAP flap * front panel status LEDS * front panel display * water cooling?"
- moved on the sheet: M?, TH1, TH2, TH?
