File: schematics/anchor/anchor.kicad_sch (KiCad schematic)
At the start: 103 parts, among them M1 Crossflow_Fan, M2 Crossflow_Fan, M3 Fan_4pin, M4 Fan_4pin, M5 Fan_4pin, M6 Fan_4pin, SW1 SW_SPST, SW2 SW_SPST, U1 e-CAM20_CU0230, U2 OLED_HDMI_USB_Display, U3 Overhub_7-Port_USB_3.0_MTT_Hub, U4 Beacon_Regulator, U5 BTT_Octopus_Max_EZ, U6 5160T_Plus, U7 5160T_Plus, U8 5160T_Plus, U9 5160T_Plus

Commit message: Connect additional nets
Parts:
- gave numbers to parts that had none: 84
Connections:
- net +48V: now also U5. (GND)
- net BED_HEATER+: now also U5. (GND)
- net BED_HEATER-: now also U5. (GND)
- net BED_THERM_0: now also U5. (GND)
- net BED_THERM_1: now also U5. (GND)
- net CH_CIRC_FAN+: now also U5. (GND)
- net CH_CIRC_FAN-: now also U5. (GND)
- net CH_HEATER+: now also U5. (GND)
- net CH_HEATER-: now also U5. (GND)
- net HE_HEATER+: now also U5. (GND)
- net HE_HEATER-: now also U5. (GND)
- net HE_THERM_0: now also U5. (GND)
- net HE_THERM_1: now also U5. (GND)
- net at J1.1 (L): now also F1.2
- net at J1.2 (N): now also SW7.1
- net at U27.: now also SW7.4, T1.1 (V-), U29.1 (1/L1)
- net CH_FAN+ renamed CH_HE_FAN+
- net CH_HE_FAN+: now also U5. (GND)
- net CH_FAN- renamed CH_HE_FAN-
- net CH_HE_FAN-: now also U5. (GND)
- net CH_FAN_ALARM renamed CH_HE_FAN_ALARM
- net CH_HE_FAN_ALARM: now also U5. (GND)
- net CH_THERM_0 renamed CH_HE_THERM_0
- net CH_HE_THERM_0: now also U5. (GND)
- net CH_THERM_1 renamed CH_HE_THERM_1
- net CH_HE_THERM_1: now also U5. (GND)
- no-connect marks 87 -> 90
Other:
- note added: "Octopus"
- note added: "TODO * microcontrollers * stepper drivers * therm board * CPAP fan * front panel status LEDS * water cooling? * toolhead leds? * contactor/SSR indicators"
- note removed: "TODO * microcontrollers * stepper drivers * CPAP fan * front panel status LEDS * water cooling? * toolhead leds?"
- moved on the sheet: F1, F2, F3, F4, F5, F6, F7, F8, J1, M15, M16, M17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

Commit message: Finish first draft of schematic
Parts:
- removed J1: IEC_60320_C14_Receptacle, symbol Connector:IEC_60320_C14_Receptacle
- removed M10: Motor_Z2, symbol Motor:Stepper_Motor_bipolar
- removed M11: Motor_X0, symbol Motor:Stepper_Motor_bipolar
- removed M12, M13, M14, M19: Motor_E0, symbol Motor:Stepper_Motor_bipolar
- removed M17, M18: Fan, symbol Motor:Fan_3pin
- removed M7: Motor_CPAP_Flap, symbol Motor:Stepper_Motor_bipolar
- removed M8: Motor_Z0, symbol Motor:Stepper_Motor_bipolar
- removed M9: Motor_Z1, symbol Motor:Stepper_Motor_bipolar
- removed SW3, SW4: SW_DPST, symbol Switch:SW_DPST
- removed T1: Meanwell_UHP-200-5, symbol jmatt:UHP-200-24
- removed T2: Meanwell_UHP-200-48, symbol jmatt:UHP-200-24
- removed T3: Meanwell_UHP-200-24, symbol jmatt:UHP-200-24
- removed U10, U11, U14, U15, U18, U19, U22, U23: Disco_On_A_Stick_XXL, symbol jmatt:Disco_On_A_Stick_XXL
- removed U32, U36, U38: ~, symbol jmatt:Murrelektronik_Diode_Zener_Suppressor
- added F9: XXA, symbol Device:Fuse
- added J4: Screw_Terminal_01x01, symbol Connector:Screw_Terminal_01x01
- added J5: IEC_60320_C14_Receptacle, symbol jmatt:IEC_60320_C14_Receptacle
- added M20: Motor_X0, symbol jmatt:Stepper_Motor_bipolar_rotated
- added M21: Motor_Y0, symbol jmatt:Stepper_Motor_bipolar_rotated
- added M22: Motor_X1, symbol jmatt:Stepper_Motor_bipolar_rotated
- added M23: Motor_Y1, symbol jmatt:Stepper_Motor_bipolar_rotated
- added M24: Motor_Z2, symbol jmatt:Stepper_Motor_bipolar_rotated
- added M25: Motor_Z1, symbol jmatt:Stepper_Motor_bipolar_rotated
- added M26: Motor_Z0, symbol jmatt:Stepper_Motor_bipolar_rotated
- added M27: Motor_CPAP_Flap, symbol jmatt:Stepper_Motor_bipolar_rotated
- added M28: Motor_E0, symbol jmatt:Stepper_Motor_bipolar_rotated
- added M7, M8: Fan, symbol jmatt:Fan_3pin_Alarm
- added SW8: SW_DPST, symbol Switch:SW_DPST
- added T1: Meanwell UHP-200-5, symbol jmatt:Meanwell_UHP-200-5
- added T2: Meanwell UHP-200-48, symbol jmatt:Meanwell_UHP-200-48
- added T3: Meanwell UHP-200-24, symbol jmatt:Meanwell_UHP-200-24
- added U32: Neopixel_Strip, symbol jmatt:Neopixel_Strip
- added U41: ThermEX26, symbol jmatt:ThermEX26
- added U42, U43, U44: ~, symbol jmatt:Murrelektronik_26051_Diode_Zener_Suppressor
Connections:
- net CH_HE_FAN_ALARM is gone; now on net Y_ENDSTOP: U5. (GND)
- net +24V: now also T3.2 (V+)
- net +48V: now also T2.2 (V+)
- net +5V: now also SW8.3, T1.2 (V+); no longer U5. (GND)
- net 120VAC_L_SWITCHED: no longer U29.2 (2/T1)
- net 120VAC_N_SWITCHED: no longer U29.4 (4/T2)
- net BED_CONTACTOR+: now also U44.1 (+)
- net BED_CONTACTOR-: now also U44.2 (-)
- net CHAMBER_LED+: now also U5. (GND)
- net CHAMBER_LED-: now also U5. (GND)
- net CH_CONTACTOR+: now also U42.1 (+)
- net CH_CONTACTOR-: now also U42.2 (-)
- net CH_HE_FAN+: now also M7.2 (+), M8.2 (+)
- net CH_HE_FAN-: now also M7.1 (-), M8.1 (-)
- net EBAY_EXHAUST_THERM_0: now also U41. (GND)
- net EBAY_EXHAUST_THERM_1: now also U41. (GND)
- net EBAY_INTAKE_THERM_0: now also U41. (GND)
- net EBAY_INTAKE_THERM_1: now also U41. (GND)
- net EBAY_LED+: now also U5. (GND)
- net EBAY_LED-: now also U5. (GND)
- net GND: now also T1.1 (V-), T2.1 (V-), T3.1 (V-), U32.3 (GND), U41. (GND)
- net HE_CONTACTOR+: now also U43.1 (+)
- net HE_CONTACTOR-: now also U43.2 (-)
- net LOWER_CH_THERM_0_0: now also U41. (GND)
- net LOWER_CH_THERM_0_1: now also U41. (GND)
- net LOWER_CH_THERM_1_0: now also U41. (GND)
- net LOWER_CH_THERM_1_1: now also U41. (GND)
- net LOWER_CH_THERM_2_0: now also U41. (GND)
- net LOWER_CH_THERM_2_1: now also U41. (GND)
- net MOTOR_CPAP_FLAP_A1: now also M27.4
- net MOTOR_CPAP_FLAP_A2: now also M27.3
- net MOTOR_CPAP_FLAP_B1: now also M27.1
- net MOTOR_CPAP_FLAP_B2: now also M27.2 (-)
- net MOTOR_E0_A1: now also M28.4
- net MOTOR_E0_A2: now also M28.3
- net MOTOR_E0_B1: now also M28.1
- net MOTOR_E0_B2: now also M28.2 (-)
- net MOTOR_E0_THERM_0: now also U41. (GND)
- net MOTOR_E0_THERM_1: now also U41. (GND)
- net MOTOR_X0_A1: now also M20.4
- net MOTOR_X0_A2: now also M20.3
- net MOTOR_X0_B1: now also M20.1
- net MOTOR_X0_B2: now also M20.2 (-)
- net MOTOR_X0_THERM_0: now also U41. (GND)
- net MOTOR_X0_THERM_1: now also U41. (GND)
- net MOTOR_X1_A1: now also M22.4
- net MOTOR_X1_A2: now also M22.3
- net MOTOR_X1_B1: now also M22.1
- net MOTOR_X1_B2: now also M22.2 (-)
- net MOTOR_X1_THERM_0: now also U41. (GND)
- net MOTOR_X1_THERM_1: now also U41. (GND)
- net MOTOR_Y0_A1: now also M21.4
- net MOTOR_Y0_A2: now also M21.3
- net MOTOR_Y0_B1: now also M21.1
- net MOTOR_Y0_B2: now also M21.2 (-)
- net MOTOR_Y0_THERM_0: now also U41. (GND)
- net MOTOR_Y0_THERM_1: now also U41. (GND)
- net MOTOR_Y1_A1: now also M23.4
- net MOTOR_Y1_A2: now also M23.3
- net MOTOR_Y1_B1: now also M23.1
- net MOTOR_Y1_B2: now also M23.2 (-)
- net MOTOR_Y1_THERM_0: now also U41. (GND)
- net MOTOR_Y1_THERM_1: now also U41. (GND)
- net MOTOR_Z0_A1: now also M26.4
- net MOTOR_Z0_A2: now also M26.3
- net MOTOR_Z0_B1: now also M26.1
- net MOTOR_Z0_B2: now also M26.2 (-)
- net MOTOR_Z0_THERM_0: now also U41. (GND)
- net MOTOR_Z0_THERM_1: now also U41. (GND)
- net MOTOR_Z1_A1: now also M25.4
- net MOTOR_Z1_A2: now also M25.3
- net MOTOR_Z1_B1: now also M25.1
- net MOTOR_Z1_B2: now also M25.2 (-)
- net MOTOR_Z1_THERM_0: now also U41. (GND)
- net MOTOR_Z1_THERM_1: now also U41. (GND)
- net MOTOR_Z2_A1: now also M24.4
- net MOTOR_Z2_A2: now also M24.3
- net MOTOR_Z2_B1: now also M24.1
- net MOTOR_Z2_B2: now also M24.2 (-)
- net MOTOR_Z2_THERM_0: now also U41. (GND)
- net MOTOR_Z2_THERM_1: now also U41. (GND)
- net THERMX_D+: now also U41. (GND)
- net THERMX_D-: now also U41. (GND)
- net UPPER_CH_THERM_0_0: now also U41. (GND)
- net UPPER_CH_THERM_0_1: now also U41. (GND)
- net UPPER_CH_THERM_1_0: now also U41. (GND)
- net UPPER_CH_THERM_1_1: now also U41. (GND)
- net UPPER_CH_THERM_2_0: now also U41. (GND)
- net UPPER_CH_THERM_2_1: now also U41. (GND)
- net VBUS: now also U3.6 (VBUS), U39. (VBUS), U5. (GND), U41. (GND)
- net at F1.2: now also J5.4 (L)
- net at SW7.1: now also F9.1
- net at U27.: now also U28.1, U29.A1
- net at SW7.4, U27., U29.1 (1/L1): now also T1.1 (V-)
- net at SW7.2, U28.2, U29.3 (3/L2)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: now also T1.2 (V+)
- net CHASSIS renamed Earth
- net Earth: now also J4.1 (Pin_1), J5.5 (PE), T1.3 (PE), T2.3 (PE), T3.3 (PE)
- new net: SW8.2, U32.2 (DIN)
- new net: SW8.4, U32.1 (+5VDC)
- new net: F9.2, J5.6 (N)
- new net: T2.1 (V-), T3.1 (V-), U29.2 (2/T1)
- new net: T2.2 (V+), T3.2 (V+), U29.4 (4/T2)
- new net CH_HE_FAN_1_ALARM: M7.3 (Alarm), U5. (GND)
- new net CH_HE_FAN_2_ALARM: M8.3 (Alarm), U5. (GND)
- new net STATUS_NEO: SW8.1, U5. (GND)
- no-connect marks 90 -> 115
Other:
- note added: "Chamber Misc"
- note added: "Chassis"
- note added: "E-Bay Misc"
- note added: "TODO * CPAP fan * contactor/SSR LED indicators * water cooling? * toolhead leds? * find final value of all XXA fuses * research more about fan rotor alarm integration"
- note added: "Themistor Board"
- note removed: "//TODO"
- note removed: "TODO * microcontrollers * stepper drivers * therm board * CPAP fan * front panel status LEDS * water cooling? * toolhead leds? * contactor/SSR indicators"
- moved on the sheet: F1, F2, F3, F4, F5, F6, F7, F8, M1, M15, M16, M2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
